Commit message: ROS 2 Jazzy migration

File: pilz_tutorial/urdf/my_first_application.xacro (robot description, xacro)
@@ -26,4 +26,6 @@
   <!-- instantiate the robot -->
   <xacro:prbt prefix="prbt_"/>
+  <!-- instantiate ros2_control for manipulator -->
+  <xacro:prbt_ros2_control prefix="prbt_"/>
   <link name="world">
     <visual>
@@ -69,10 +71,8 @@
     <child link="prbt_base_link"/>
   </joint>
-  <joint name="pnoz_joint" type="prismatic">
+  <joint name="pnoz_joint" type="fixed">
     <origin rpy="0 0 0" xyz="0 -0.5 0.115"/>
     <parent link="prbt_base_link"/>
     <child link="pnoz"/>
-    <axis xyz="0 0 1"/>
-    <limit effort="1000.0" lower="-1" upper="1" velocity="1"/>
   </joint>
   <!-- TCP -->
@@ -91,4 +91,6 @@
     <!-- instantiate gripper -->
     <xacro:prbt_gripper parent="$(arg robot_prefix)flange" />
+    <!-- instantiate ros2_control for gripper -->
+    <xacro:prbt_gripper_ros2_control prefix="$(arg robot_prefix)"/>
     <!-- Add gripper brackets -->
     <xacro:include filename="$(find prbt_support)/urdf/simple_gripper_brackets.urdf.xacro" />

File: prbt_grippers/prbt_pg70_support/config/pg70.srdf.xacro (robot description, xacro)
@@ -58,5 +58,30 @@
     <disable_collisions link1="${prefix}gripper_finger_right_link_bracket" link2="${prefix}link_5" reason="Never" />
     <disable_collisions link1="${prefix}gripper_palm_link" link2="${prefix}link_2" reason="Never" />
+    <disable_collisions link1="${prefix}gripper_palm_link" link2="${prefix}link_3" reason="Never" />
+    <disable_collisions link1="${prefix}gripper_palm_link" link2="${prefix}link_4" reason="Never" />
     <disable_collisions link1="${prefix}gripper_palm_link" link2="${prefix}link_5" reason="Never" />
+    <disable_collisions link1="${prefix}gripper_finger_left_link" link2="${prefix}link_3" reason="Never" />
+    <disable_collisions link1="${prefix}gripper_finger_left_link" link2="${prefix}link_4" reason="Never" />
+    <disable_collisions link1="${prefix}gripper_finger_left_link_bracket" link2="${prefix}link_3" reason="Never" />
+    <disable_collisions link1="${prefix}gripper_finger_left_link_bracket" link2="${prefix}link_4" reason="Never" />
+    <disable_collisions link1="${prefix}gripper_finger_right_link" link2="${prefix}link_3" reason="Never" />
+    <disable_collisions link1="${prefix}gripper_finger_right_link" link2="${prefix}link_4" reason="Never" />
+    <disable_collisions link1="${prefix}gripper_finger_right_link_bracket" link2="${prefix}link_3" reason="Never" />
+    <disable_collisions link1="${prefix}gripper_finger_right_link_bracket" link2="${prefix}link_4" reason="Never" />
+    <!-- gripper vs link_1, link_2, base_link - physically unreachable -->
+    <disable_collisions link1="${prefix}gripper_palm_link" link2="${prefix}link_1" reason="Never" />
+    <disable_collisions link1="${prefix}gripper_palm_link" link2="${prefix}base_link" reason="Never" />
+    <disable_collisions link1="${prefix}gripper_finger_left_link" link2="${prefix}link_1" reason="Never" />
+    <disable_collisions link1="${prefix}gripper_finger_left_link" link2="${prefix}link_2" reason="Never" />
+    <disable_collisions link1="${prefix}gripper_finger_left_link" link2="${prefix}base_link" reason="Never" />
+    <disable_collisions link1="${prefix}gripper_finger_right_link" link2="${prefix}link_1" reason="Never" />
+    <disable_collisions link1="${prefix}gripper_finger_right_link" link2="${prefix}link_2" reason="Never" />
+    <disable_collisions link1="${prefix}gripper_finger_right_link" link2="${prefix}base_link" reason="Never" />
+    <disable_collisions link1="${prefix}gripper_finger_left_link_bracket" link2="${prefix}link_1" reason="Never" />
+    <disable_collisions link1="${prefix}gripper_finger_left_link_bracket" link2="${prefix}link_2" reason="Never" />
+    <disable_collisions link1="${prefix}gripper_finger_left_link_bracket" link2="${prefix}base_link" reason="Never" />
+    <disable_collisions link1="${prefix}gripper_finger_right_link_bracket" link2="${prefix}link_1" reason="Never" />
+    <disable_collisions link1="${prefix}gripper_finger_right_link_bracket" link2="${prefix}link_2" reason="Never" />
+    <disable_collisions link1="${prefix}gripper_finger_right_link_bracket" link2="${prefix}base_link" reason="Never" />
   </xacro:macro>
   <!-- instantiate gripper -->

File: prbt_moveit_config/config/prbt.srdf.xacro (robot description, xacro)
@@ -7,5 +7,5 @@
   <!--VIRTUAL JOINT: Purpose: this element defines a virtual joint between a robot link and an
                      external frame of reference (considered fixed with respect to the robot)-->
-  <virtual_joint name="FixedBase" type="fixed" parent_frame="$(arg prefix)base_link" child_link="world" />
+  <virtual_joint name="FixedBase" type="fixed" parent_frame="world" child_link="world" />
   <!-- robot manipulator -->
   <xacro:include filename="$(find prbt_moveit_config)/config/prbt_manipulator.srdf.xacro" />

File: prbt_support/urdf/prbt_macro.xacro (robot description, xacro)
@@ -42,4 +42,5 @@
     </link>
     <!-- arm 1 joint -->
+    <!-- NOTE: velocity moderately elevated for simulation (mock_components). Real hardware: 1.57 rad/s -->
     <joint name="${prefix}joint_1" type="revolute">
       <origin xyz="0 0 ${L0}" rpy="0 0 -${pi}"/>
@@ -47,5 +48,5 @@
       <child link="${prefix}link_1"/>
       <axis xyz="0 0 1"/>
-      <limit effort="370" velocity="1.57" lower="-2.96706" upper="2.96706"/>
+      <limit effort="370" velocity="5.0" lower="-2.96706" upper="2.96706"/>
       <dynamics damping="15.0" friction="11" />
     </joint>
@@ -88,5 +89,5 @@
       <child link="${prefix}link_2"/>
       <axis xyz="0 0 1"/>
-      <limit effort="370" velocity="1.57" lower="-2.53073" upper="2.53073"/>
+      <limit effort="370" velocity="5.0" lower="-2.53073" upper="2.53073"/>
       <dynamics damping="12.0" friction="10.0" />
     </joint>
@@ -122,5 +123,5 @@
       <child link="${prefix}link_3"/>
       <axis xyz="0 0 1"/>
-      <limit effort="176" velocity="1.57" lower="-2.35620" upper="2.35620"/>
+      <limit effort="176" velocity="5.0" lower="-2.35620" upper="2.35620"/>
       <dynamics damping="4.5" friction="4.5" />
     </joint>
@@ -162,5 +163,5 @@
       <child link="${prefix}link_4"/>
       <axis xyz="0 0 1" />
-      <limit effort="176" velocity="1.57" lower="-2.96706" upper="2.96706"/>
+      <limit effort="176" velocity="5.0" lower="-2.96706" upper="2.96706"/>
       <dynamics damping="4.2" friction="3.8" />
     </joint>
@@ -196,5 +197,5 @@
       <child link="${prefix}link_5"/>
       <axis xyz="0 0 1" />
-      <limit effort="41.6" velocity="1.57" lower="-2.96706" upper="2.96706" />
+      <limit effort="41.6" velocity="200.0" lower="-2.96706" upper="2.96706" />
       <dynamics damping="1.5" friction="3.5" />
     </joint>
@@ -248,5 +249,5 @@
       <child link="${prefix}flange"/>
       <axis xyz="0 0 1" />
-      <limit effort="20.1" velocity="1.57" lower="-3.12414" upper="3.12414" />
+      <limit effort="20.1" velocity="5.0" lower="-3.12414" upper="3.12414" />
       <dynamics damping="4.5" friction="7.0" />
     </joint>
@@ -271,5 +272,5 @@
       </collision>
     </link>
-    <!-- ROS-Industrial 'base' frame: base_link to robot world coordinate sytem transform -->
+    <!-- ROS-Industrial 'base' frame: base_link to robot world coordinate system transform -->
     <link name="${prefix}base" />
     <joint name="${prefix}base_link-base" type="fixed">
@@ -285,114 +286,55 @@
       <child link="${prefix}tool0" />
     </joint>
-    <!-- transmissions for gazebo -->
-    <transmission name="${prefix}joint_1_trans">
-      <type>transmission_interface/SimpleTransmission</type>
+  </xacro:macro>
+  <!-- ros2_control macro for the manipulator -->
+  <xacro:macro name="prbt_ros2_control" params="prefix">
+    <ros2_control name="prbt_manipulator" type="system">
+      <hardware>
+        <plugin>mock_components/GenericSystem</plugin>
+      </hardware>
       <joint name="${prefix}joint_1">
-        <hardwareInterface>hardware_interface/PositionJointInterface</hardwareInterface>
-      </joint>
-      <actuator name="${prefix}joint_1_motor"/>
-    </transmission>
-    <transmission name="${prefix}joint_2_trans">
-      <type>transmission_interface/SimpleTransmission</type>
+        <command_interface name="position"/>
+        <state_interface name="position"><param name="initial_value">0.0</param></state_interface>
+        <state_interface name="velocity"/>
+      </joint>
       <joint name="${prefix}joint_2">
-        <hardwareInterface>hardware_interface/PositionJointInterface</hardwareInterface>
-      </joint>
-      <actuator name="${prefix}joint_2_motor"/>
-    </transmission>
-    <transmission name="${prefix}joint_3_trans">
-      <type>transmission_interface/SimpleTransmission</type>
+        <command_interface name="position"/>
+        <state_interface name="position"><param name="initial_value">0.0</param></state_interface>
+        <state_interface name="velocity"/>
+      </joint>
       <joint name="${prefix}joint_3">
-        <hardwareInterface>hardware_interface/PositionJointInterface</hardwareInterface>
-      </joint>
-      <actuator name="${prefix}joint_3_motor"/>
-    </transmission>
-    <transmission name="${prefix}joint_4_trans">
-      <type>transmission_interface/SimpleTransmission</type>
+        <command_interface name="position"/>
+        <state_interface name="position"><param name="initial_value">0.0</param></state_interface>
+        <state_interface name="velocity"/>
+      </joint>
       <joint name="${prefix}joint_4">
-        <hardwareInterface>hardware_interface/PositionJointInterface</hardwareInterface>
-      </joint>
-      <actuator name="${prefix}joint_4_motor"/>
-    </transmission>
-    <transmission name="${prefix}joint_5_trans">
-      <type>transmission_interface/SimpleTransmission</type>
+        <command_interface name="position"/>
+        <state_interface name="position"><param name="initial_value">0.0</param></state_interface>
+        <state_interface name="velocity"/>
+      </joint>
       <joint name="${prefix}joint_5">
-        <hardwareInterface>hardware_interface/PositionJointInterface</hardwareInterface>
-      </joint>
-      <actuator name="${prefix}joint_5_motor"/>
-    </transmission>
-    <transmission name="${prefix}joint_6_trans">
-      <type>transmission_interface/SimpleTransmission</type>
+        <command_interface name="position"/>
+        <state_interface name="position"><param name="initial_value">0.0</param></state_interface>
+        <state_interface name="velocity"/>
+      </joint>
       <joint name="${prefix}joint_6">
-        <hardwareInterface>hardware_interface/PositionJointInterface</hardwareInterface>
-      </joint>
-      <actuator name="${prefix}joint_6_motor"/>
-    </transmission>
-    <gazebo>
-      <plugin name="gazebo_ros_control" filename="libgazebo_ros_control.so" >
-        <robotNamespace>prbt</robotNamespace>
-        <robotSimType>gazebo_ros_control/DefaultRobotHWSim</robotSimType>
-        <legacyModeNS>false</legacyModeNS> <!-- Only used from ros-kinetic-gazebo-ros-control 2.5.18 -->
-      </plugin>
-    </gazebo>
-    <gazebo reference="${prefix}joint_1">
-      <provideFeedback>true</provideFeedback>
-    </gazebo>
-    <gazebo>
-      <plugin name="ft_sensor" filename="libgazebo_ros_ft_sensor.so">
-	<updateRate>100.0</updateRate>
-	<topicName>prbt/ft_sensor/joint_1</topicName>
-	<jointName>${prefix}joint_1</jointName>
-      </plugin>
-    </gazebo>
-    <gazebo reference="${prefix}joint_2">
-      <provideFeedback>true</provideFeedback>
-    </gazebo>
-    <gazebo>
-      <plugin name="ft_sensor" filename="libgazebo_ros_ft_sensor.so">
-	<updateRate>100.0</updateRate>
-	<topicName>prbt/ft_sensor/joint_2</topicName>
-	<jointName>${prefix}joint_2</jointName>
-      </plugin>
-    </gazebo>
-    <gazebo reference="${prefix}joint_3">
-      <provideFeedback>true</provideFeedback>
-    </gazebo>
-    <gazebo>
-      <plugin name="ft_sensor" filename="libgazebo_ros_ft_sensor.so">
-	<updateRate>100.0</updateRate>
-	<topicName>prbt/ft_sensor/joint_3</topicName>
-	<jointName>${prefix}joint_3</jointName>
-      </plugin>
-    </gazebo>
-    <gazebo reference="${prefix}joint_4">
-      <provideFeedback>true</provideFeedback>
-    </gazebo>
-    <gazebo>
-      <plugin name="ft_sensor" filename="libgazebo_ros_ft_sensor.so">
-	<updateRate>100.0</updateRate>
-	<topicName>prbt/ft_sensor/joint_4</topicName>
-	<jointName>${prefix}joint_4</jointName>
-      </plugin>
-    </gazebo>
-    <gazebo reference="${prefix}joint_5">
-      <provideFeedback>true</provideFeedback>
-    </gazebo>
-    <gazebo>
-      <plugin name="ft_sensor" filename="libgazebo_ros_ft_sensor.so">
-	<updateRate>100.0</updateRate>
-	<topicName>prbt/ft_sensor/joint_5</topicName>
-	<jointName>${prefix}joint_5</jointName>
-      </plugin>
-    </gazebo>
-    <gazebo reference="${prefix}joint_6">
-      <provideFeedback>true</provideFeedback>
-    </gazebo>
-    <gazebo>
-      <plugin name="ft_sensor" filename="libgazebo_ros_ft_sensor.so">
-	<updateRate>100.0</updateRate>
-	<topicName>prbt/ft_sensor/joint_6</topicName>
-	<jointName>${prefix}joint_6</jointName>
-      </plugin>
-    </gazebo>
+        <command_interface name="position"/>
+        <state_interface name="position"><param name="initial_value">0.0</param></state_interface>
+        <state_interface name="velocity"/>
+      </joint>
+    </ros2_control>
+  </xacro:macro>
+  <!-- ros2_control macro for the gripper -->
+  <xacro:macro name="prbt_gripper_ros2_control" params="prefix">
+    <ros2_control name="prbt_gripper" type="system">
+      <hardware>
+        <plugin>mock_components/GenericSystem</plugin>
+      </hardware>
+      <joint name="${prefix}gripper_finger_left_joint">
+        <command_interface name="position"/>
+        <state_interface name="position"><param name="initial_value">0.0</param></state_interface>
+        <state_interface name="velocity"/>
+      </joint>
+    </ros2_control>
   </xacro:macro>
 </robot>
