Commit message: fix gripper

File: schunk_description/urdf/pg70/pg70.urdf.xacro (robot description, xacro)
@@ -61,5 +61,6 @@
       <child link="${name}_finger_left_link" />
       <axis xyz="0 1 0" />
-      <limit effort="10" lower="-0.001" upper="0.061" velocity="2.0"/>
+      <!-- <limit effort="10" lower="-0.001" upper="0.061" velocity="2.0"/> -->
+      <limit effort="10" lower="-0.0001" upper="0.05" velocity="2.0"/>
     </joint>
     <link name="${name}_finger_left_link">
@@ -92,5 +93,6 @@
       <axis xyz="0 -1 0" />
       <mimic joint="${name}_finger_left_joint" multiplier="1" offset="0"/>
-      <limit effort="10" lower="-0.001" upper="0.061" velocity="2.0"/>
+      <!-- <limit effort="10" lower="-0.001" upper="0.061" velocity="2.0"/> -->
+      <limit effort="10" lower="-0.0001" upper="0.05" velocity="2.0"/>
     </joint>
     <link name="${name}_finger_right_link">
